File: tutorial.kicad_pcb (KiCad board)
At the start: 2 copper layers, 77.8 x 38.1 mm, 24 parts, among them SW1 SW_Push, U1 ATmega32U4-AU, Y1 16MHz

Commit message: fix pcb layout
Routing:
- net COL1: track 19.0 -> 54.9 mm
- net ROW0: track 19.7 -> 48.9 mm
- net ROW1: track 20.3 -> 46.7 mm
- net COL0: track 19.0 -> 31.0 mm
- added copper zone on B.Cu, net GND
Changed lines of the file:
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@@
   (general
     (thickness 1.6)
-    (drawings 7)
-    (tracks 196)
+    (drawings 8)
+    (tracks 218)
     (zones 0)
     (modules 24)
@@
     (visible_elements FFFFFF7F)
     (pcbplotparams
-      (layerselection 0x010fc_ffffffff)
-      (usegerberextensions false)
+      (layerselection 0x010f0_ffffffff)
+      (usegerberextensions true)
       (usegerberattributes true)
       (usegerberadvancedattributes true)
-      (creategerberjobfile true)
+      (creategerberjobfile false)
       (excludeedgelayer true)
       (linewidth 0.100000)
@@
       (plotinvisibletext false)
       (padsonsilk false)
-      (subtractmaskfromsilk false)
+      (subtractmaskfromsilk true)
       (outputformat 1)
       (mirror false)
-      (drillshape 1)
+      (drillshape 0)
       (scaleselection 1)
-      (outputdirectory ""))
+      (outputdirectory "Gerbers"))
   )
   (net 0 "")
@@
     (fp_line (start 1.68 0.95) (end 1.68 -0.95) (layer B.CrtYd) (width 0.05))
     (fp_line (start 1.68 -0.95) (end -1.68 -0.95) (layer B.CrtYd) (width 0.05))
-    (pad 2 smd roundrect (at 0.9125 0 90) (size 1.025 1.4) (layers B.Cu B.Paste B.Mask) (roundrect_rratio 0.243902)
+    (pad 2 smd roundrect (at 0.9125 0 90) (size 1.025 1.4) (layers B.Cu B.Paste B.Mask) (roundrect_rratio 0.2439014634146341)
       (net 20 "Net-(R4-Pad2)"))
-    (pad 1 smd roundrect (at -0.9125 0 90) (size 1.025 1.4) (layers B.Cu B.Paste B.Mask) (roundrect_rratio 0.243902)
+    (pad 1 smd roundrect (at -0.9125 0 90) (size 1.025 1.4) (layers B.Cu B.Paste B.Mask) (roundrect_rratio 0.2439014634146341)
       (net 1 GND))
     (model ${KISYS3DMOD}/Resistor_SMD.3dshapes/R_0805_2012Metric.wrl
@@
     (fp_line (start 1.68 0.95) (end 1.68 -0.95) (layer B.CrtYd) (width 0.05))
     (fp_line (start 1.68 -0.95) (end -1.68 -0.95) (layer B.CrtYd) (width 0.05))
-    (pad 2 smd roundrect (at 0.9125 0 270) (size 1.025 1.4) (layers B.Cu B.Paste B.Mask) (roundrect_rratio 0.243902)
+    (pad 2 smd roundrect (at 0.9125 0 270) (size 1.025 1.4) (layers B.Cu B.Paste B.Mask) (roundrect_rratio 0.2439014634146341)
       (net 19 "Net-(R3-Pad2)"))
-    (pad 1 smd roundrect (at -0.9125 0 270) (size 1.025 1.4) (layers B.Cu B.Paste B.Mask) (roundrect_rratio 0.243902)
+    (pad 1 smd roundrect (at -0.9125 0 270) (size 1.025 1.4) (layers B.Cu B.Paste B.Mask) (roundrect_rratio 0.2439014634146341)
       (net 2 +5V))
     (model ${KISYS3DMOD}/Resistor_SMD.3dshapes/R_0805_2012Metric.wrl
@@
     (fp_line (start 1.68 0.95) (end 1.68 -0.95) (layer B.CrtYd) (width 0.05))
     (fp_line (start 1.68 -0.95) (end -1.68 -0.95) (layer B.CrtYd) (width 0.05))
-    (pad 2 smd roundrect (at 0.9125 0 90) (size 1.025 1.4) (layers B.Cu B.Paste B.Mask) (roundrect_rratio 0.243902)
+    (pad 2 smd roundrect (at 0.9125 0 90) (size 1.025 1.4) (layers B.Cu B.Paste B.Mask) (roundrect_rratio 0.2439014634146341)
       (net 17 D+))
-    (pad 1 smd roundrect (at -0.9125 0 90) (size 1.025 1.4) (layers B.Cu B.Paste B.Mask) (roundrect_rratio 0.243902)
+    (pad 1 smd roundrect (at -0.9125 0 90) (size 1.025 1.4) (layers B.Cu B.Paste B.Mask) (roundrect_rratio 0.2439014634146341)
       (net 18 "Net-(R2-Pad1)"))
     (model ${KISYS3DMOD}/Resistor_SMD.3dshapes/R_0805_2012Metric.wrl
@@
     (fp_line (start 1.68 0.95) (end 1.68 -0.95) (layer B.CrtYd) (width 0.05))
     (fp_line (start 1.68 -0.95) (end -1.68 -0.95) (layer B.CrtYd) (width 0.05))
-    (pad 2 smd roundrect (at 0.9125 0 90) (size 1.025 1.4) (layers B.Cu B.Paste B.Mask) (roundrect_rratio 0.243902)
+    (pad 2 smd roundrect (at 0.9125 0 90) (size 1.025 1.4) (layers B.Cu B.Paste B.Mask) (roundrect_rratio 0.2439014634146341)
       (net 15 D-))
-    (pad 1 smd roundrect (at -0.9125 0 90) (size 1.025 1.4) (layers B.Cu B.Paste B.Mask) (roundrect_rratio 0.243902)
+    (pad 1 smd roundrect (at -0.9125 0 90) (size 1.025 1.4) (layers B.Cu B.Paste B.Mask) (roundrect_rratio 0.2439014634146341)
       (net 16 "Net-(R1-Pad1)"))
     (model ${KISYS3DMOD}/Resistor_SMD.3dshapes/R_0805_2012Metric.wrl
@@
     )
   )
+  (gr_line (start 117.475 97.63125) (end 117.475 130.96875) (layer Edge.Cuts) (width 0.05))
   (gr_arc (start 42.06875 130.96875) (end 39.6875 130.96875) (angle -90) (layer Edge.Cuts) (width 0.05))
   (gr_arc (start 42.06875 97.63125) (end 42.06875 95.25) (angle -90) (layer Edge.Cuts) (width 0.05))
@@
   (segment (start 98.4875 106.425) (end 99.21875 107.15625) (width 0.25) (layer B.Cu) (net 7))
   (segment (start 96.8375 106.425) (end 98.4875 106.425) (width 0.25) (layer B.Cu) (net 7))
+  (segment (start 88.9625 114.3) (end 96.8375 106.425) (width 0.25) (layer B.Cu) (net 7))
+  (segment (start 88.9 114.3) (end 88.9625 114.3) (width 0.25) (layer B.Cu) (net 7))
+  (segment (start 88.434348 114.765652) (end 88.9 114.3) (width 0.25) (layer B.Cu) (net 7))
+  (segment (start 82.3636 114.765652) (end 88.434348 114.765652) (width 0.25) (layer B.Cu) (net 7))
+  (segment (start 73.16875 119.85) (end 74.60625 119.85) (width 0.25) (layer B.Cu) (net 7))
+  (segment (start 77.273002 119.85625) (end 82.3636 114.765652) (width 0.25) (layer B.Cu) (net 7))
+  (segment (start 74.6125 119.85625) (end 77.273002 119.85625) (width 0.25) (layer B.Cu) (net 7))
+  (segment (start 74.60625 119.85) (end 74.6125 119.85625) (width 0.25) (layer B.Cu) (net 7))
   (segment (start 113.0375 100.275) (end 115.8875 103.125) (width 0.25) (layer B.Cu) (net 8))
   (segment (start 110.45 100.275) (end 113.0375 100.275) (width 0.25) (layer B.Cu) (net 8))
@@
   (segment (start 114.3625 127) (end 115.8875 125.475) (width 0.25) (layer B.Cu) (net 9))
   (segment (start 100.0125 127) (end 114.3625 127) (width 0.25) (layer B.Cu) (net 9))
+  (segment (start 96.8375 125.475) (end 96.8375 125.4125) (width 0.25) (layer B.Cu) (net 9))
+  (segment (start 96.8375 125.4125) (end 95.25 127) (width 0.25) (layer B.Cu) (net 9))
+  (segment (start 95.25 127) (end 84.1375 127) (width 0.25) (layer B.Cu) (net 9))
+  (segment (start 84.1375 127) (end 79.375 122.2375) (width 0.25) (layer B.Cu) (net 9))
+  (segment (start 79.3625 122.25) (end 73.16875 122.25) (width 0.25) (layer B.Cu) (net 9))
+  (segment (start 79.375 122.2375) (end 79.3625 122.25) (width 0.25) (layer B.Cu) (net 9))
   (segment (start 93.9875 119.325) (end 96.8375 122.175) (width 0.25) (layer B.Cu) (net 10))
   (segment (start 91.4 119.325) (end 93.9875 119.325) (width 0.25) (layer B.Cu) (net 10))
@@
   (segment (start 110.45 119.325) (end 113.0375 119.325) (width 0.25) (layer B.Cu) (net 11))
   (segment (start 85.09 102.235) (end 85.09 121.285) (width 0.25) (layer F.Cu) (net 13))
+  (segment (start 84.925 121.45) (end 85.09 121.285) (width 0.25) (layer B.Cu) (net 13))
+  (segment (start 73.16875 121.45) (end 84.925 121.45) (width 0.25) (layer B.Cu) (net 13))
   (segment (start 104.14 102.235) (end 104.14 121.285) (width 0.25) (layer F.Cu) (net 14))
+  (segment (start 77.115662 120.65) (end 82.55 115.215662) (width 0.25) (layer B.Cu) (net 14))
+  (segment (start 73.16875 120.65) (end 77.115662 120.65) (width 0.25) (layer B.Cu) (net 14))
+  (segment (start 82.55 115.215662) (end 96.715588 115.215662) (width 0.25) (layer B.Cu) (net 14))
+  (segment (start 96.715588 115.215662) (end 96.8375 115.09375) (width 0.25) (layer B.Cu) (net 14))
+  (segment (start 97.94875 115.09375) (end 104.14 121.285) (width 0.25) (layer B.Cu) (net 14))
+  (segment (start 96.8375 115.09375) (end 97.94875 115.09375) (width 0.25) (layer B.Cu) (net 14))
   (segment (start 55.5625 112.83125) (end 53.85625 112.83125) (width 0.25) (layer B.Cu) (net 19))
   (segment (start 53.85625 112.83125) (end 53.18125 113.50625) (width 0.25) (layer B.Cu) (net 19))
@@
   (segment (start 73.2 124.61875) (end 73.16875 124.65) (width 0.25) (layer B.Cu) (net 20))
   (segment (start 76.2 124.61875) (end 73.2 124.61875) (width 0.25) (layer B.Cu) (net 20))
+  (zone (net 1) (net_name GND) (layer B.Cu) (hatch edge 0.508)
+    (connect_pads (clearance 0.508))
+    (min_thickness 0.254)
+    (fill yes (arc_segments 32) (thermal_gap 0.508) (thermal_bridge_width 0.508))
+    (polygon
+      (pts
+        (xy 79.375 133.35) (xy 39.6875 133.35) (xy 39.6875 95.25) (xy 79.375 95.25)
+      )
+    )
+  )
 )
